File: Hardware/pro-micro_hub.kicad_sch (KiCad schematic)
At the start: 9 parts, among them J12 I2C_M, J8 Parallel_F, U11 ATmega32U4-M, U12 ATtiny88-A

Commit message: added SPI port on the schematic, added .history in .gitignore
Parts:
- added SPI_F: SPI_F, symbol Connector_Generic:Conn_01x05
- UART_F: renamed from USB_F; value USB_F -> UART_F
- USB_F: renamed from UART_F; value UART_F -> USB_F
Connections:
- net +5V: now also SPI_F.4 (Pin_4)
- net GND: now also SPI_F.5 (Pin_5)
- net MISO: now also SPI_F.2 (Pin_2)
- net MOSI: now also SPI_F.1 (Pin_1)
- net SCK: now also SPI_F.3 (Pin_3)
